File: macro-deck-pcb/macro-deck-pcb.kicad_sch (KiCad schematic)
At the start: 0 parts

Commit message: started schematic
started schematic design - pi pico and usb-c circutry (because i hate micro-usb lol) sketched it out using some circutry design and footprints/symbols from adafruit product 4090 bc im lazy and have never implemented a usb c port directly on my project before.
Parts:
- added A1: RaspberryPi_Pico, Module:RaspberryPi_Pico_SMD, symbol MCU_Module:RaspberryPi_Pico_Extensive
- added R1, R2: 5.1k, symbol Device:R
- added X1: USB_C, macro-deck-imported:USB_C_CUSB31-CFM2AX-01-X, symbol macro-deck-imported:USB_C
Connections:
- new net: R2.1, X1.B5 (CC2)
- new net: R1.1, X1.A5 (CC1)
- new net: A1.13 (GND), A1.18 (GND), A1.23 (GND), A1.28 (GND), A1.3 (GND), A1.38 (GND), A1.8 (GND), A1.D2 (GND)
- new net USB_D+: A1.TP3 (USB_DP), X1.A6 (D+), X1.B6 (D+)
- new net USB_D-: A1.TP2 (USB_DM), X1.A7 (D-), X1.B7 (D-)
- new net USB_GND: A1.TP1 (USB_GND), R1.2, R2.2, X1.A1B12 (GND), X1.B1A12 (GND)
- new net VBUS: A1.40 (VBUS), X1.A4B9 (VBUS), X1.B4A9 (VBUS)
